Commit message: Imported upstream version '1.0.2' of 'upstream'

File: flir_ptu_description/urdf/ptu5.urdf.xacro (robot description, xacro)
@@ -127,5 +127,5 @@
       <parent link="${name}_tilt_link"/>
       <child link="${name}_mount_link"/>
-      <origin xyz="0 0 0" rpy="0 0 0" />
+      <origin xyz="0 0 0.0757" rpy="0 0 0" />
     </joint>
     <!--
